File: hardware/motor/pxia--motor--controller-encoder/pxia--motor--controller-encoder.kicad_sch (KiCad schematic)
At the start: 7 parts

Commit message: updated schematics + footprint
Changed lines of the file:
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@@
   )
   (text "mounting holes aligned to SMCI12 PCB mounting holes.\n22MM hole could also be reduced to 5MM shaft diameter."
-    (at 153.67 127 0)
+    (at 185.42 123.19 0)
     (effects (font (size 1.27 1.27)) (justify left bottom))
   )

Commit message: finished schematics and most of pcb layout
Parts:
- removed H?: Ø 22MM, symbol Mechanical:MountingHole
- removed J?: IDC-Connector, symbol Connector_Generic:Conn_02x06_Odd_Even
- added C1: 100nF, Capacitor_SMD:C_0603_1608Metric, symbol Device:C_Small
- added C2: 1nF, Capacitor_SMD:C_0603_1608Metric, symbol Device:C_Small
- added J1: IDC(CTRL>), Connector_Molex:Molex_Nano-Fit_105314-xx12_2x06_P2.50mm_Horizontal, symbol Connector_Generic:Conn_02x06_Top_Bottom
- added J2: GPIO+PWR, Connector_Molex:Molex_Nano-Fit_105314-xx16_2x08_P2.50mm_Horizontal, symbol Connector_Generic:Conn_02x08_Top_Bottom
- added R1: 10K, Resistor_SMD:R_0603_1608Metric, symbol Device:R_Small
- H1, H2, H3, H4: renamed from H?; footprint (none) -> MountingHole:MountingHole_3.2mm_M3
- U1: renamed from U?; value A1101LLHL -> MT8512AT; footprint Package_TO_SOT_SMD:SOT-23W -> Package_TO_SOT_SMD:SOT-23_Handsoldering
Connections:
- net +5V: now also C1.2, J1.6 (Pin_6), J2.1 (Pin_1), J2.5 (Pin_5), J2.6 (Pin_6), R1.1
- net ANALOG_IN: now also J1.11 (Pin_11), J2.8 (Pin_8)
- net GND: now also C1.1, C2.2, J1.7 (Pin_7), J2.12 (Pin_12), J2.13 (Pin_13), J2.16 (Pin_16)
- net INPUT_1: now also C2.1, J1.5 (Pin_5), J2.9 (Pin_9), R1.2
- net INPUT_2: now also J1.4 (Pin_4), J2.2 (Pin_2)
- net INPUT_3: now also J1.3 (Pin_3), J2.10 (Pin_10)
- net INPUT_4: now also J1.2 (Pin_2), J2.3 (Pin_3)
- net INPUT_5: now also J1.1 (Pin_1), J2.11 (Pin_11)
- net INPUT_6: now also J1.12 (Pin_12), J2.4 (Pin_4)
- net OUTPUT_1: now also J1.10 (Pin_10), J2.14 (Pin_14)
- net OUTPUT_2: now also J1.9 (Pin_9), J2.7 (Pin_7)
- net OUTPUT_3: now also J1.8 (Pin_8), J2.15 (Pin_15)
Other:
- note added: ">>> FROM CONTROLLER"
- note added: "MFR.Part # MT8512AT"
- note added: "PROTOTYPING AREA >>>"
- note added: "SOT-23-3"
- note removed: "@TODO maybe use a different connector type … maybe IDC @TODO maybe reorder the pins"
- note removed: "A1101LLHL is an SMD SOT-23W package version. maybe use a THT component?"
- note removed: "FROM CONTROLLER >>>"

Commit message: added PicoW, finished PCB layout
Parts:
- C1: value 100nF -> (none); footprint Capacitor_SMD:C_0603_1608Metric -> (none); LCSC (none) -> C14663
- C2: LCSC (none) -> C1588
- R1: LCSC (none) -> C25804
- U1: LCSC (none) -> C879601
Changed lines of the file:
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@@
     (effects (font (size 1.27 1.27)) (justify left bottom))
+  )
+  (symbol (lib_id "power:GND") (at 166.37 99.06 0) (unit 1)
+    (in_bom yes) (on_board yes) (fields_autoplaced)
+    (property "Reference" "#PWR0106" (id 0) (at 166.37 105.41 0)
+      (effects (font (size 1.27 1.27)) hide)
+    )
+    (property "Value" "GND" (id 1) (at 166.37 104.14 0))
+    (property "Footprint" "" (id 2) (at 166.37 99.06 0)
+      (effects (font (size 1.27 1.27)) hide)
+    )
+    (property "Datasheet" "" (id 3) (at 166.37 99.06 0)
+      (effects (font (size 1.27 1.27)) hide)
+    )
+    (pin "1")
   )
   (symbol (lib_id "power:+5V") (at 80.01 48.26 0) (unit 1)
@@
       (effects (font (size 1.27 1.27)) hide)
     )
+    (property "LCSC" "C25804" (id 4) (at 102.87 99.06 0)
+      (effects (font (size 1.27 1.27)) hide)
+    )
     (pin "1")
     (pin "2")
@@
       (effects (font (size 1.27 1.27)) (justify right))
     )
-    (property "Value" "100nF" (id 1) (at 67.31 114.2935 0)
-      (effects (font (size 1.27 1.27)) (justify right))
-    )
-    (property "Footprint" "Capacitor_SMD:C_0603_1608Metric" (id 2) (at 69.85 113.03 0)
+    (property "Value" "" (id 1) (at 67.31 114.2935 0)
+      (effects (font (size 1.27 1.27)) (justify right))
+    )
+    (property "Footprint" "" (id 2) (at 69.85 113.03 0)
       (effects (font (size 1.27 1.27)) hide)
     )
     (property "Datasheet" "~" (id 3) (at 69.85 113.03 0)
+      (effects (font (size 1.27 1.27)) hide)
+    )
+    (property "LCSC" "C14663" (id 4) (at 69.85 113.03 0)
       (effects (font (size 1.27 1.27)) hide)
     )
@@
     (pin "9")
   )
+  (symbol (lib_id "power:+5V") (at 154.94 99.06 180) (unit 1)
+    (in_bom yes) (on_board yes)
+    (property "Reference" "#PWR0105" (id 0) (at 154.94 95.25 0)
+      (effects (font (size 1.27 1.27)) hide)
+    )
+    (property "Value" "+5V" (id 1) (at 154.94 104.14 0))
+    (property "Footprint" "" (id 2) (at 154.94 99.06 0)
+      (effects (font (size 1.27 1.27)) hide)
+    )
+    (property "Datasheet" "" (id 3) (at 154.94 99.06 0)
+      (effects (font (size 1.27 1.27)) hide)
+    )
+    (pin "1")
+  )
   (symbol (lib_id "Device:C_Small") (at 100.33 113.03 0) (unit 1)
     (in_bom yes) (on_board yes) (fields_autoplaced)
@@
     )
     (property "Datasheet" "~" (id 3) (at 100.33 113.03 0)
+      (effects (font (size 1.27 1.27)) hide)
+    )
+    (property "LCSC" "C1588" (id 4) (at 100.33 113.03 0)
       (effects (font (size 1.27 1.27)) hide)
     )
@@
       (effects (font (size 1.27 1.27)) hide)
     )
+    (property "LCSC" "C879601" (id 4) (at 90.17 106.68 0)
+      (effects (font (size 1.27 1.27)) hide)
+    )
     (pin "1")
     (pin "2")
@@
     (pin "1")
   )
+  (symbol (lib_id "power:PWR_FLAG") (at 154.94 99.06 0) (unit 1)
+    (in_bom yes) (on_board yes) (fields_autoplaced)
+    (property "Reference" "#FLG0101" (id 0) (at 154.94 97.155 0)
+      (effects (font (size 1.27 1.27)) hide)
+    )
+    (property "Value" "PWR_FLAG" (id 1) (at 154.94 93.98 0))
+    (property "Footprint" "" (id 2) (at 154.94 99.06 0)
+      (effects (font (size 1.27 1.27)) hide)
+    )
+    (property "Datasheet" "~" (id 3) (at 154.94 99.06 0)
+      (effects (font (size 1.27 1.27)) hide)
+    )
+    (pin "1")
+  )
+  (symbol (lib_id "power:PWR_FLAG") (at 166.37 99.06 0) (unit 1)
+    (in_bom yes) (on_board yes) (fields_autoplaced)
+    (property "Reference" "#FLG0102" (id 0) (at 166.37 97.155 0)
+      (effects (font (size 1.27 1.27)) hide)
+    )
+    (property "Value" "PWR_FLAG" (id 1) (at 166.37 93.98 0))
+    (property "Footprint" "" (id 2) (at 166.37 99.06 0)
+      (effects (font (size 1.27 1.27)) hide)
+    )
+    (property "Datasheet" "~" (id 3) (at 166.37 99.06 0)
+      (effects (font (size 1.27 1.27)) hide)
+    )
+    (pin "1")
+  )
   (symbol (lib_id "power:GND") (at 105.41 68.58 0) (unit 1)
     (in_bom yes) (on_board yes) (fields_autoplaced)
@@
   )
   (symbol_instances
+    (path "/e6b41409-6620-4b5b-a599-b37644ff2228"
+      (reference "#FLG0101") (unit 1) (value "PWR_FLAG") (footprint "")
+    )
+    (path "/e93c60ce-d3bc-4bae-b80e-61594d75b6f4"
+      (reference "#FLG0102") (unit 1) (value "PWR_FLAG") (footprint "")
+    )
     (path "/202a2a60-27a6-4809-9d3a-8adaeea463ba"
       (reference "#PWR0101") (unit 1) (value "+5V") (footprint "")
@@
       (reference "#PWR0104") (unit 1) (value "+5V") (footprint "")
     )
+    (path "/97df6bf6-41ba-405e-8d66-58a907c7652f"
+      (reference "#PWR0105") (unit 1) (value "+5V") (footprint "")
+    )
+    (path "/0b114951-e6e0-4d0d-bfd1-7bbccded62a9"
+      (reference "#PWR0106") (unit 1) (value "GND") (footprint "")
+    )
     (path "/7787030c-1f3e-482b-94d0-35e959f33ad4"

Commit message: updated PCB and schematics
Parts:
- C2: value 1nF -> (none); footprint Capacitor_SMD:C_0603_1608Metric -> (none)
- H1, H2, H3, H4: value M3 -> (none); footprint MountingHole:MountingHole_3.2mm_M3 -> (none)
- J1: value IDC(CTRL>) -> (none); footprint Connector_Molex:Molex_Nano-Fit_105314-xx12_2x06_P2.50mm_Horizontal -> (none); LCSC (none) -> DNF
- J2: value GPIO+PWR -> (none); footprint Connector_Molex:Molex_Nano-Fit_105314-xx16_2x08_P2.50mm_Horizontal -> (none); LCSC (none) -> DNF
- R1: value 10K -> (none); footprint Resistor_SMD:R_0603_1608Metric -> (none)
- U1: value MT8512AT -> (none); footprint Package_TO_SOT_SMD:SOT-23_Handsoldering -> (none)
Changed lines of the file:
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@@
       (effects (font (size 1.27 1.27)) (justify right))
     )
-    (property "Value" "10K" (id 1) (at 105.41 100.3299 0)
-      (effects (font (size 1.27 1.27)) (justify right))
-    )
-    (property "Footprint" "Resistor_SMD:R_0603_1608Metric" (id 2) (at 102.87 99.06 0)
+    (property "Value" "" (id 1) (at 105.41 100.3299 0)
+      (effects (font (size 1.27 1.27)) (justify right))
+    )
+    (property "Footprint" "" (id 2) (at 102.87 99.06 0)
       (effects (font (size 1.27 1.27)) hide)
     )
@@
       (effects (font (size 1.27 1.27)) (justify left))
     )
-    (property "Value" "M3" (id 1) (at 168.91 121.9199 0)
-      (effects (font (size 1.27 1.27)) (justify left))
-    )
-    (property "Footprint" "MountingHole:MountingHole_3.2mm_M3" (id 2) (at 166.37 120.65 0)
+    (property "Value" "" (id 1) (at 168.91 121.9199 0)
+      (effects (font (size 1.27 1.27)) (justify left))
+    )
+    (property "Footprint" "" (id 2) (at 166.37 120.65 0)
       (effects (font (size 1.27 1.27)) hide)
     )
@@
       (effects (font (size 1.27 1.27)) (justify left))
     )
-    (property "Value" "M3" (id 1) (at 156.21 115.5699 0)
-      (effects (font (size 1.27 1.27)) (justify left))
-    )
-    (property "Footprint" "MountingHole:MountingHole_3.2mm_M3" (id 2) (at 153.67 114.3 0)
+    (property "Value" "" (id 1) (at 156.21 115.5699 0)
+      (effects (font (size 1.27 1.27)) (justify left))
+    )
+    (property "Footprint" "" (id 2) (at 153.67 114.3 0)
       (effects (font (size 1.27 1.27)) hide)
     )
@@
       (effects (font (size 1.27 1.27)) (justify left))
     )
-    (property "Value" "M3" (id 1) (at 156.21 121.9199 0)
-      (effects (font (size 1.27 1.27)) (justify left))
-    )
-    (property "Footprint" "MountingHole:MountingHole_3.2mm_M3" (id 2) (at 153.67 120.65 0)
+    (property "Value" "" (id 1) (at 156.21 121.9199 0)
+      (effects (font (size 1.27 1.27)) (justify left))
+    )
+    (property "Footprint" "" (id 2) (at 153.67 120.65 0)
       (effects (font (size 1.27 1.27)) hide)
     )
@@
       (effects (font (size 1.27 1.27)) (justify left))
     )
-    (property "Value" "M3" (id 1) (at 168.91 115.5699 0)
-      (effects (font (size 1.27 1.27)) (justify left))
-    )
-    (property "Footprint" "MountingHole:MountingHole_3.2mm_M3" (id 2) (at 166.37 114.3 0)
+    (property "Value" "" (id 1) (at 168.91 115.5699 0)
+      (effects (font (size 1.27 1.27)) (justify left))
+    )
+    (property "Footprint" "" (id 2) (at 166.37 114.3 0)
       (effects (font (size 1.27 1.27)) hide)
     )
@@
     (in_bom yes) (on_board yes)
     (property "Reference" "J2" (id 0) (at 172.72 48.26 0))
-    (property "Value" "GPIO+PWR" (id 1) (at 172.72 71.12 0))
-    (property "Footprint" "Connector_Molex:Molex_Nano-Fit_105314-xx16_2x08_P2.50mm_Horizontal" (id 2) (at 171.45 58.42 0)
+    (property "Value" "" (id 1) (at 172.72 71.12 0))
+    (property "Footprint" "" (id 2) (at 171.45 58.42 0)
       (effects (font (size 1.27 1.27)) hide)
     )
     (property "Datasheet" "~" (id 3) (at 171.45 58.42 0)
+      (effects (font (size 1.27 1.27)) hide)
+    )
+    (property "LCSC" "DNF" (id 4) (at 171.45 58.42 0)
       (effects (font (size 1.27 1.27)) hide)
     )
@@
       (effects (font (size 1.27 1.27)) (justify left))
     )
-    (property "Value" "1nF" (id 1) (at 102.87 114.3062 0)
-      (effects (font (size 1.27 1.27)) (justify left))
-    )
-    (property "Footprint" "Capacitor_SMD:C_0603_1608Metric" (id 2) (at 100.33 113.03 0)
+    (property "Value" "" (id 1) (at 102.87 114.3062 0)
+      (effects (font (size 1.27 1.27)) (justify left))
+    )
+    (property "Footprint" "" (id 2) (at 100.33 113.03 0)
       (effects (font (size 1.27 1.27)) hide)
     )
@@
     (in_bom yes) (on_board yes)
     (property "Reference" "J1" (id 0) (at 90.17 49.53 0))
-    (property "Value" "IDC(CTRL>)" (id 1) (at 90.17 67.31 0))
-    (property "Footprint" "Connector_Molex:Molex_Nano-Fit_105314-xx12_2x06_P2.50mm_Horizontal" (id 2) (at 88.9 59.69 0)
+    (property "Value" "" (id 1) (at 90.17 67.31 0))
+    (property "Footprint" "" (id 2) (at 88.9 59.69 0)
       (effects (font (size 1.27 1.27)) hide)
     )
     (property "Datasheet" "~" (id 3) (at 88.9 59.69 0)
+      (effects (font (size 1.27 1.27)) hide)
+    )
+    (property "LCSC" "DNF" (id 4) (at 88.9 59.69 0)
       (effects (font (size 1.27 1.27)) hide)
     )
@@
       (effects (font (size 1.27 1.27)) (justify right))
     )
-    (property "Value" "MT8512AT" (id 1) (at 83.82 107.9499 0)
-      (effects (font (size 1.27 1.27)) (justify right))
-    )
-    (property "Footprint" "Package_TO_SOT_SMD:SOT-23_Handsoldering" (id 2) (at 90.17 115.57 0)
+    (property "Value" "" (id 1) (at 83.82 107.9499 0)
+      (effects (font (size 1.27 1.27)) (justify right))
+    )
+    (property "Footprint" "" (id 2) (at 90.17 115.57 0)
       (effects (font (size 1.27 1.27) italic) (justify left) hide)
     )
